Commit message: change colors

File: example_robot.urdf.xacro (robot description, xacro)
@@ -26,6 +26,6 @@
                 <box size="2.5 1.5 0.1" />
             </geometry>
-            <material name="green">
-                <color rgba="0.2 1 0.2 1"/>
+            <material name="purple">
+                <color rgba="0.9 .1 0.8 1"/>
             </material>
         </visual>

Commit message: change shape

File: example_robot.urdf.xacro (robot description, xacro)
@@ -24,5 +24,5 @@
             <origin xyz="0 0 0.05" rpy="0 0 0"/>
             <geometry>
-                <box size="2.5 1.5 0.1" />
+                <box size="1.5 1.5 0.1" />
             </geometry>
             <material name="purple">
@@ -90,6 +90,6 @@
     <!-- - The visual/collision origin is set to halfway along the length (similar to the box), but also with a rotation (again using the mathematical features). -->
     <!--   This is because the cylinder extends along the Z axis by default, but we want it to be along the X axis (when the joint is at 0) -->
-    <xacro:property name="arm_length" value="2" />
-    <xacro:property name="arm_radius" value="0.02" />
+    <xacro:property name="arm_length" value="1" />
+    <xacro:property name="arm_radius" value="0.04" />
     <link name="arm_link">
         <visual>

File: example_robot_xacroed.urdf (robot description, URDF)
Before this commit: robot robot, 5 links, 4 joints
Links:
- link arm_link: geometry collision cylinder length=1 radius=0.04; visual cylinder length=1 radius=0.04
- link base_link: geometry collision box size=2.5 1.5 0.1; visual box size=1.5 1.5 0.1
Joints:
- joint camera_joint: origin xyz=2 0 0.095 rpy=0 0 0 -> xyz=1 0 0.11499999999999999 rpy=0 0 0
